File: _autosave-zotbins_2025_wrover_pcb.kicad_sch (KiCad schematic)
At the start: 41 parts, among them J1 FFC2B28-24-G, J10 DCJ200-10-A-XX-K_REVA, J2 DCJ200-10-A-XX-K_REVA, J3 HC-SR04_Screw_Terminal_01x04, J4 HX711_Screw_Terminal_01x04, J5 Main_Servo_Screw_Terminal_01x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, J6 Conn_01x30_Pin, J7 SG_Servo_Screw_Terminal_01x03, J8 BB_Receiver_Screw_Terminal_01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, J9 BB_Transmitter_Screw_Terminal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

Commit message: basically the final version; just final adjustments with labeling and silkscreen needed. Traces, all components are all set.
Other:
- note added: "Camera Power Step Down"
- note added: "Main Power"
- note added: "Servo Power"
Changed lines of the file:
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@@
+		)
+	)
+	(text "Main Power"
+		(exclude_from_sim no)
+		(at 30.226 143.002 0)
+		(effects
+			(font
+				(size 1.27 1.27)
+			)
 		)
 	)
@@
 		(effects
 			(font
+				(size 1.27 1.27)
+			)
+		)
+	)
+	(text "Camera Power Step Down"
+		(exclude_from_sim no)
+		(at 113.03 106.934 0)
+		(effects
+			(font
+				(size 1.27 1.27)
+			)
+		)
+	)
+	(text "Servo Power"
+		(exclude_from_sim no)
+		(at 30.226 108.966 0)
+		(effects
+			(font
