File: zotbins_2025_wrover_pcb.kicad_pcb (KiCad board)
At the start: 2 copper layers, 125 x 125 mm, 40 parts, among them J1 Conn_01x28_Pin, J2 DCJ200-10-A-XX-K_REVA, J3 HC-SR04_Screw_Terminal_01x04, J4 HX711_Screw_Terminal_01x05, J5 Main_Servo_Screw_Terminal_01x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, J6 Conn_01x30_Pin, J7 SG_Servo_Screw_Terminal_01x03, J8 BB_Receiver_Screw_Terminal_01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, J9 BB_Transmitter_Screw_Terminal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, U1 LM350_TO220, U2 MCP23017_SP, U3 XC6206P302MR-G, U4 XC6206P282PR-G, U5 LM7805_TO220, U6 ESP32-DEVKITC-32D

Commit message: changed hcsr04 power to 3V3 as this component changed models
Connections:
- J3 pad 4: +5V -> +3V3
Routing:
- net +5V: track 274.9 -> 262.0 mm
- net +3V3: track 544.9 -> 549.2 mm
Other:
- board text added: "3V3"
Changed lines of the file:
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@@
 			(layers "*.Cu" "*.Mask")
 			(remove_unused_layers no)
-			(net 2 "+5V")
+			(net 47 "+3V3")
 			(pinfunction "Pin_4")
 			(pintype "passive")
@@
 		)
 	)
-	(gr_text "+5V"
+	(gr_text "3V3\n"
 		(at 203.973992 119.944527 0)
 		(layer "F.SilkS")
@@
 	)
 	(gr_text "OV2640"
-		(at 165.061477 128.97526 0)
+		(at 170.059356 128.97526 0)
 		(layer "F.SilkS")
 		(effects
@@
 	)
 	(segment
-		(start 209.793475 119.051573)
-		(end 202.44272 126.402328)
-		(width 1.5)
-		(layer "F.Cu")
-		(net 2)
-	)
-	(segment
 		(start 139 140.1)
 		(end 145.842397 146.942397)
@@
 	)
 	(segment
-		(start 212.3 119.051573)
-		(end 209.793475 119.051573)
-		(width 1.5)
-		(layer "F.Cu")
-		(net 2)
-	)
-	(segment
 		(start 145.842397 146.942397)
 		(end 152.859367 146.942397)
@@
 	)
 	(segment
+		(start 215.47215 119.051573)
+		(end 216.236088 118.287635)
+		(width 1)
+		(layer "F.Cu")
+		(net 47)
+	)
+	(segment
 		(start 118.48353 105.130769)
 		(end 115.63448 105.130769)
@@
 	)
 	(segment
+		(start 216.236088 118.287635)
+		(end 216.236088 158.791248)
+		(width 1)
+		(layer "F.Cu")
+		(net 47)
+	)
+	(segment
 		(start 184.405735 132.669462)
 		(end 184.405735 131.296051)
@@
 	)
 	(segment
+		(start 212.3 119.051573)
+		(end 215.47215 119.051573)
+		(width 1)
+		(layer "F.Cu")
+		(net 47)
+	)
+	(segment
 		(start 196.770269 130.737169)
 		(end 193.986037 130.737169)
@@
 	(segment
 		(start 216.236088 97.79678)
-		(end 216.236088 158.791248)
+		(end 216.236088 118.287635)
 		(width 1)
 		(layer "F.Cu")

Commit message: fixed net name ambiguity on schematic
Connections:
- R1 pad 2: /GPIO_SDA -> /GPIO_SCK
- R2 pad 2: /GPIO_SCK -> /GPIO_SDA
- U2 pad 12: /GPIO_SDA -> /GPIO_SCK
- U2 pad 13: /GPIO_SCK -> /GPIO_SDA
- U6 pad J2-12: /GPIO_SDA -> /GPIO_SCK
- U6 pad J2-15: /GPIO_SCK -> /GPIO_SDA
Routing:
- net /GPIO_SDA: track 47.4 -> 51.2 mm
- net /GPIO_SCK: track 51.2 -> 47.4 mm
Changed lines of the file:
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@@
 			(layers "*.Cu" "*.Mask")
 			(remove_unused_layers no)
-			(net 43 "/GPIO_SDA")
+			(net 42 "/GPIO_SCK")
 			(pinfunction "IO14")
 			(pintype "bidirectional")
@@
 			(layers "*.Cu" "*.Mask")
 			(remove_unused_layers no)
-			(net 42 "/GPIO_SCK")
+			(net 43 "/GPIO_SDA")
 			(pinfunction "IO13")
 			(pintype "bidirectional")
@@
 			(layers "*.Cu" "*.Mask")
 			(remove_unused_layers no)
-			(net 43 "/GPIO_SDA")
+			(net 42 "/GPIO_SCK")
 			(pintype "passive")
 		)
@@
 			(layers "*.Cu" "*.Mask")
 			(remove_unused_layers no)
-			(net 43 "/GPIO_SDA")
+			(net 42 "/GPIO_SCK")
 			(pinfunction "SCK")
 			(pintype "input")
@@
 			(layers "*.Cu" "*.Mask")
 			(remove_unused_layers no)
-			(net 42 "/GPIO_SCK")
+			(net 43 "/GPIO_SDA")
 			(pinfunction "SDA")
 			(pintype "bidirectional")
@@
 			(net 66 "/STROBE")
 			(pinfunction "Pin_1")
-			(pintype "passive")
+			(pintype "passive+no_connect")
 		)
 		(pad "2" smd rect
@@
 			(net 69 "/AGND")
 			(pinfunction "Pin_2")
-			(pintype "passive")
+			(pintype "passive+no_connect")
 		)
 		(pad "3" smd rect
@@
 			(net 68 "/PWDN")
 			(pinfunction "Pin_8")
-			(pintype "passive")
+			(pintype "passive+no_connect")
 		)
 		(pad "9" smd rect
@@
 			(net 67 "/DGND")
 			(pinfunction "Pin_15")
-			(pintype "passive")
+			(pintype "passive+no_connect")
 		)
 		(pad "16" smd rect
@@
 			(layers "*.Cu" "*.Mask")
 			(remove_unused_layers no)
-			(net 42 "/GPIO_SCK")
+			(net 43 "/GPIO_SDA")
 			(pintype "passive")
 		)
@@
 	)
 	(segment
-		(start 122.5 101.1)
-		(end 122.5 102.7)
+		(start 129.4 95.215)
+		(end 133.315 95.215)
 		(width 0.5)
 		(layer "F.Cu")
@@
 	)
 	(segment
-		(start 138.7 105.7)
-		(end 142.1 102.3)
+		(start 140.3 95.9)
+		(end 141.1 95.1)
 		(width 0.5)
 		(layer "F.Cu")
@@
 	)
 	(segment
-		(start 151.252145 99.7)
-		(end 148.452145 96.9)
+		(start 140.3 100.9)
+		(end 140.3 95.9)
 		(width 0.5)
 		(layer "F.Cu")
@@
 	)
 	(segment
-		(start 129.4 97.755)
-		(end 132.055 97.755)
+		(start 134.6 96.5)
+		(end 134.6 103)
 		(width 0.5)
 		(layer "F.Cu")
@@
 	)
 	(segment
-		(start 128.345 97.755)
-		(end 129.4 97.755)
+		(start 134.6 103)
+		(end 135.2 103.6)
 		(width 0.5)
 		(layer "F.Cu")
@@
 	)
 	(segment
-		(start 127 103.3)
-		(end 127.75 102.55)
+		(start 135.2 103.6)
+		(end 137.6 103.6)
 		(width 0.5)
 		(layer "F.Cu")
@@
 	)
 	(segment
-		(start 142.1 97.7)
-		(end 142.9 96.9)
+		(start 147.7 95.1)
+		(end 150.72 92.08)
 		(width 0.5)
 		(layer "F.Cu")
@@
 	)
 	(segment
-		(start 123.1 103.3)
-		(end 127 103.3)
+		(start 133.315 95.215)
+		(end 134.6 96.5)
 		(width 0.5)
 		(layer "F.Cu")
@@
 	)
 	(segment
-		(start 142.1 102.3)
-		(end 142.1 97.7)
+		(start 141.1 95.1)
+		(end 147.7 95.1)
 		(width 0.5)
 		(layer "F.Cu")
@@
 	)
 	(segment
-		(start 142.9 96.9)
-		(end 148.452145 96.9)
+		(start 129.265 95.08)
+		(end 129.4 95.215)
 		(width 0.5)
 		(layer "F.Cu")
@@
 	)
 	(segment
-		(start 127.75 98.35)
-		(end 128.345 97.755)
+		(start 137.6 103.6)
+		(end 140.3 100.9)
 		(width 0.5)
 		(layer "F.Cu")
@@
 	)
 	(segment
-		(start 132.055 97.755)
-		(end 132.8 98.5)
+		(start 150.72 92.08)
+		(end 152.95 92.08)
 		(width 0.5)
 		(layer "F.Cu")
@@
 	)
 	(segment
-		(start 122.5 102.7)
-		(end 123.1 103.3)
+		(start 127.185 95.215)
+		(end 125.85 96.55)
 		(width 0.5)
-		(layer "F.Cu")
+		(layer "B.Cu")
 		(net 42)
 	)
 	(segment
-		(start 134.3 105.7)
-		(end 138.7 105.7)
+		(start 125.85 96.55)
+		(end 125.85 101.08)
 		(width 0.5)
-		(layer "F.Cu")
+		(layer "B.Cu")
 		(net 42)
 	)
 	(segment
-		(start 132.8 104.2)
-		(end 134.3 105.7)
+		(start 129.4 95.215)
+		(end 127.185 95.215)
 		(width 0.5)
-		(layer "F.Cu")
+		(layer "B.Cu")
 		(net 42)
 	)
 	(segment
-		(start 132.8 98.5)
-		(end 132.8 104.2)
+		(start 122.5 101.1)
+		(end 122.5 102.7)
 		(width 0.5)
 		(layer "F.Cu")
-		(net 42)
+		(net 43)
 	)
 	(segment
-		(start 127.75 102.55)
-		(end 127.75 98.35)
+		(start 138.7 105.7)
+		(end 142.1 102.3)
 		(width 0.5)
 		(layer "F.Cu")
-		(net 42)
+		(net 43)
 	)
 	(segment
-		(start 152.95 99.7)
-		(end 151.252145 99.7)
+		(start 151.252145 99.7)
+		(end 148.452145 96.9)
 		(width 0.5)
 		(layer "F.Cu")
-		(net 42)
+		(net 43)
 	)
 	(segment
-		(start 129.4 95.215)
-		(end 133.315 95.215)
+		(start 129.4 97.755)
+		(end 132.055 97.755)
 		(width 0.5)
 		(layer "F.Cu")
@@
 	)
 	(segment
-		(start 140.3 95.9)
-		(end 141.1 95.1)
+		(start 128.345 97.755)
+		(end 129.4 97.755)
 		(width 0.5)
 		(layer "F.Cu")
@@
 	)
 	(segment
-		(start 140.3 100.9)
-		(end 140.3 95.9)
+		(start 127 103.3)
+		(end 127.75 102.55)
 		(width 0.5)
 		(layer "F.Cu")
@@
 	)
 	(segment
-		(start 134.6 96.5)
-		(end 134.6 103)
+		(start 142.1 97.7)
+		(end 142.9 96.9)
 		(width 0.5)
 		(layer "F.Cu")
@@
 	)
 	(segment
-		(start 134.6 103)
-		(end 135.2 103.6)
+		(start 123.1 103.3)
+		(end 127 103.3)
 		(width 0.5)
 		(layer "F.Cu")
@@
 	)
 	(segment
-		(start 135.2 103.6)
-		(end 137.6 103.6)
+		(start 142.1 102.3)
+		(end 142.1 97.7)
 		(width 0.5)
 		(layer "F.Cu")
@@
 	)
 	(segment
-		(start 147.7 95.1)
-		(end 150.72 92.08)
+		(start 142.9 96.9)
+		(end 148.452145 96.9)
 		(width 0.5)
 		(layer "F.Cu")
@@
 	)
 	(segment
-		(start 133.315 95.215)
-		(end 134.6 96.5)
+		(start 127.75 98.35)
+		(end 128.345 97.755)
 		(width 0.5)
 		(layer "F.Cu")
@@
 	)
 	(segment
-		(start 141.1 95.1)
-		(end 147.7 95.1)
+		(start 132.055 97.755)
+		(end 132.8 98.5)
 		(width 0.5)
 		(layer "F.Cu")
@@
 	)
 	(segment
-		(start 129.265 95.08)
-		(end 129.4 95.215)
+		(start 122.5 102.7)
+		(end 123.1 103.3)
 		(width 0.5)
 		(layer "F.Cu")
@@
 	)
 	(segment
-		(start 137.6 103.6)
-		(end 140.3 100.9)
+		(start 134.3 105.7)
+		(end 138.7 105.7)
 		(width 0.5)
 		(layer "F.Cu")
@@
 	)
 	(segment
-		(start 150.72 92.08)
-		(end 152.95 92.08)
+		(start 132.8 104.2)
+		(end 134.3 105.7)
 		(width 0.5)
 		(layer "F.Cu")
@@
 	)
 	(segment
-		(start 127.185 95.215)
-		(end 125.85 96.55)
+		(start 132.8 98.5)
+		(end 132.8 104.2)
 		(width 0.5)
-		(layer "B.Cu")
+		(layer "F.Cu")
 		(net 43)
 	)
 	(segment
-		(start 125.85 96.55)
-		(end 125.85 101.08)
+		(start 127.75 102.55)
+		(end 127.75 98.35)
 		(width 0.5)
-		(layer "B.Cu")
+		(layer "F.Cu")
 		(net 43)
 	)
 	(segment
-		(start 129.4 95.215)
-		(end 127.185 95.215)
+		(start 152.95 99.7)
+		(end 151.252145 99.7)
 		(width 0.5)
-		(layer "B.Cu")
+		(layer "F.Cu")
 		(net 43)
 	)

Commit message: ordered version + gerber
Parts:
- added J10: Conn_01x02_Pin, Connector_PinSocket_2.54mm:PinSocket_1x02_P2.54mm_Vertical, F.Cu at (155.1, 123.2)
- added J11: Hall_Screw_Terminal_01x03, TerminalBlock_4Ucon:TerminalBlock_4Ucon_1x03_P3.50mm_Vertical, F.Cu at (187.3, 41.6)
- added R8: 1k, Resistor_THT:R_Axial_DIN0207_L6.3mm_D2.5mm_P10.16mm_Horizontal, F.Cu at (151.4, 119.9)
- moved R7 11.7 mm to (201.1, 54.6), turned to 90 degrees
- moved TP4 8.70 mm to (113.0, 141.5)
- moved J2 7.63 mm to (100.7, 133.2)
- moved TP6 0.77 mm to (212.2, 50.1)
- moved C6 0.63 mm to (141.4, 126.3)
- moved C4 0.62 mm to (141.4, 118.9)
- moved TP2 0.31 mm to (150.4, 136.2)
- moved TP1 0.26 mm to (144.4, 136.1)
Connections:
- net /GPIO_12 renamed /Hall_ADC
Routing:
- net /Hall_ADC: track 127.5 -> 448.0 mm, vias 2 -> 4
- net +5V: track 262.0 -> 364.0 mm, vias 0 -> 2
- net Net-(U1-VI): track 59.3 -> 77.6 mm
- net +3V3: track 549.2 -> 540.7 mm
- net /IR: track 176.2 -> 167.9 mm
- net Net-(J10-Pin_2): track 0.00 -> 3.94 mm
- net CSI_1V2: track 66.6 -> 65.5 mm
- net /RX: track 147.8 -> 146.8 mm
- net /EN: track 160.4 -> 161.0 mm
