File: zotbins_2025_wrover_pcb.kicad_sch (KiCad schematic)
At the start: 40 parts, among them J1 Conn_01x28_Pin, J2 DCJ200-10-A-XX-K_REVA, J3 HC-SR04_Screw_Terminal_01x04, J4 HX711_Screw_Terminal_01x05, J5 Main_Servo_Screw_Terminal_01x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, J6 Conn_01x30_Pin, J7 SG_Servo_Screw_Terminal_01x03, J8 BB_Receiver_Screw_Terminal_01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, J9 BB_Transmitter_Screw_Terminal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, U1 LM350_TO220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

Commit message: ordered version + gerber
Parts:
- added J10: Conn_01x02_Pin, Connector_PinSocket_2.54mm:PinSocket_1x02_P2.54mm_Vertical, symbol Connector:Conn_01x02_Pin
- added J11: Hall_Screw_Terminal_01x03, TerminalBlock_4Ucon:TerminalBlock_4Ucon_1x03_P3.50mm_Vertical, symbol Connector:Screw_Terminal_01x03
- added R8: 1k, Resistor_THT:R_Axial_DIN0207_L6.3mm_D2.5mm_P10.16mm_Horizontal, symbol Device:R_Small
Connections:
- net +5V: now also J11.1 (Pin_1)
- net GND: now also J11.2 (Pin_2), R8.2
- net GPIO_12 renamed Hall_ADC
- net Hall_ADC: now also J10.1 (Pin_1), J11.3 (Pin_3)
- new net: J10.2 (Pin_2), R8.1
Other:
- note added: "GPIO 12 is a strapping pin. Paired with STRONG PD resistor"
- moved on the sheet: C2, J1, J3, J4, J5, J7, J8, J9, R4, R7, TP6
